File: 24Vsupply.sch (KiCad schematic (older format))
At the start: 12 parts

Commit message: Ready for tapeout
Parts:
- gave numbers to parts that had none: 12
Changed lines of the file:
@@
 $Descr A4 11693 8268
 encoding utf-8
-Sheet 3 9
+Sheet 3 10
 Title ""
 Date ""
@@
 $EndDescr
 $Comp
-L TPS55340 U?
+L TPS55340 U3
 U 1 1 5460B860
 P 4550 2750
-F 0 "U?" H 4900 3400 60  0000 C CNN
+F 0 "U3" H 4900 3400 60  0000 C CNN
 F 1 "TPS55340" H 4500 2750 60  0000 C CNN
 F 2 "" H 4500 2750 60  0000 C CNN
@@
 GNDPWR
 $Comp
-L CP2 C?
+L CP2 C14
 U 1 1 5460B955
 P 1900 2600
-F 0 "C?" H 1900 2700 40  0000 L CNN
+F 0 "C14" H 1900 2700 40  0000 L CNN
 F 1 "4.7µ" H 1906 2515 40  0000 L CNN
 F 2 "" H 1938 2450 30  0000 C CNN
@@
 $EndComp
 $Comp
-L R R?
+L R R9
 U 1 1 5460B99A
 P 3300 2550
-F 0 "R?" V 3380 2550 40  0000 C CNN
+F 0 "R9" V 3380 2550 40  0000 C CNN
 F 1 "60.4k" V 3307 2551 40  0000 C CNN
 F 2 "" V 3230 2550 30  0000 C CNN
@@
 $EndComp
 $Comp
-L C C?
+L C C16
 U 1 1 5460B9E7
 P 2800 2700
-F 0 "C?" H 2800 2800 40  0000 L CNN
+F 0 "C16" H 2800 2800 40  0000 L CNN
 F 1 "150n" H 2806 2615 40  0000 L CNN
 F 2 "" H 2838 2550 30  0000 C CNN
@@
 $EndComp
 $Comp
-L C C?
+L C C17
 U 1 1 5460BA88
 P 3150 3300
-F 0 "C?" H 3150 3400 40  0000 L CNN
+F 0 "C17" H 3150 3400 40  0000 L CNN
 F 1 "680p" H 3156 3215 40  0000 L CNN
 F 2 "" H 3188 3150 30  0000 C CNN
@@
 $EndComp
 $Comp
-L R R?
+L R R8
 U 1 1 5460BB14
 P 2800 3000
-F 0 "R?" V 2880 3000 40  0000 C CNN
+F 0 "R8" V 2880 3000 40  0000 C CNN
 F 1 "422" V 2807 3001 40  0000 C CNN
 F 2 "" V 2730 3000 30  0000 C CNN
@@
 $EndComp
 $Comp
-L C C?
+L C C15
 U 1 1 5460BBBE
 P 2400 3300
-F 0 "C?" H 2400 3400 40  0000 L CNN
+F 0 "C15" H 2400 3400 40  0000 L CNN
 F 1 "680n" H 2406 3215 40  0000 L CNN
 F 2 "" H 2438 3150 30  0000 C CNN
@@
 $EndComp
 $Comp
-L R R?
+L R R11
 U 1 1 5460BC03
 P 7200 3250
-F 0 "R?" V 7280 3250 40  0000 C CNN
+F 0 "R11" V 7280 3250 40  0000 C CNN
 F 1 "10k" V 7207 3251 40  0000 C CNN
 F 2 "" V 7130 3250 30  0000 C CNN
@@
 $EndComp
 $Comp
-L R R?
+L R R10
 U 1 1 5460BC95
 P 7200 2200
-F 0 "R?" V 7280 2200 40  0000 C CNN
+F 0 "R10" V 7280 2200 40  0000 C CNN
 F 1 "187k" V 7207 2201 40  0000 C CNN
 F 2 "" V 7130 2200 30  0000 C CNN
@@
 $EndComp
 $Comp
-L C C?
+L C C18
 U 1 1 5460BCD0
 P 7700 2900
-F 0 "C?" H 7700 3000 40  0000 L CNN
+F 0 "C18" H 7700 3000 40  0000 L CNN
 F 1 "4.7µ" H 7706 2815 40  0000 L CNN
 F 2 "" H 7738 2750 30  0000 C CNN
@@
 $EndComp
 $Comp
-L INDUCTOR L?
+L INDUCTOR L2
 U 1 1 5460BD3C
 P 4550 1800
-F 0 "L?" V 4500 1800 40  0000 C CNN
+F 0 "L2" V 4500 1800 40  0000 C CNN
 F 1 "27µ" V 4650 1800 40  0000 C CNN
 F 2 "" H 4550 1800 60  0000 C CNN
@@
 $EndComp
 $Comp
-L DIODESCH D?
+L DIODESCH D1
 U 1 1 5460BDD5
 P 6300 1800
-F 0 "D?" H 6300 1900 40  0000 C CNN
+F 0 "D1" H 6300 1900 40  0000 C CNN
 F 1 "2A" H 6300 1700 40  0000 C CNN
 F 2 "" H 6300 1800 60  0000 C CNN
