File: 5Vsupply.sch (KiCad schematic (older format))
At the start: 7 parts

Commit message: Ready for tapeout
Parts:
- gave numbers to parts that had none: 7
Changed lines of the file:
@@
 $Descr A4 11693 8268
 encoding utf-8
-Sheet 2 9
+Sheet 2 10
 Title ""
 Date ""
@@
 $EndComp
 $Comp
-L C C?
+L C C11
 U 1 1 54608AEC
 P 4300 3850
-F 0 "C?" H 4300 3950 40  0000 L CNN
+F 0 "C11" H 4300 3950 40  0000 L CNN
 F 1 "22u" H 4306 3765 40  0000 L CNN
 F 2 "" H 4338 3700 30  0000 C CNN
@@
 	4300 4050 4300 4400
 $Comp
-L C C?
+L C C12
 U 1 1 54608B55
 P 5750 3550
-F 0 "C?" V 5600 3500 40  0000 L CNN
+F 0 "C12" V 5600 3500 40  0000 L CNN
 F 1 "100n" V 5900 3450 40  0000 L CNN
 F 2 "" H 5788 3400 30  0000 C CNN
@@
 $EndComp
 $Comp
-L C C?
+L C C13
 U 1 1 54608BA0
 P 7100 3850
-F 0 "C?" H 7100 3950 40  0000 L CNN
+F 0 "C13" H 7100 3950 40  0000 L CNN
 F 1 "47u" H 7106 3765 40  0000 L CNN
 F 2 "" H 7138 3700 30  0000 C CNN
@@
 $EndComp
 $Comp
-L R R?
+L R R6
 U 1 1 54608C09
 P 6650 3550
-F 0 "R?" V 6730 3550 40  0000 C CNN
+F 0 "R6" V 6730 3550 40  0000 C CNN
 F 1 "56.2k" V 6657 3551 40  0000 C CNN
 F 2 "" V 6580 3550 30  0000 C CNN
@@
 $EndComp
 $Comp
-L R R?
+L R R7
 U 1 1 54608C56
 P 6650 4150
-F 0 "R?" V 6730 4150 40  0000 C CNN
+F 0 "R7" V 6730 4150 40  0000 C CNN
 F 1 "10k" V 6657 4151 40  0000 C CNN
 F 2 "" V 6580 4150 30  0000 C CNN
@@
 $EndComp
 $Comp
-L INDUCTOR L?
+L INDUCTOR L1
 U 1 1 54608CA7
 P 6250 3300
-F 0 "L?" V 6200 3300 40  0000 C CNN
+F 0 "L1" V 6200 3300 40  0000 C CNN
 F 1 "3.3uH" V 6350 3300 40  0000 C CNN
 F 2 "" H 6250 3300 60  0000 C CNN
@@
 Vfb
 $Comp
-L TPS563209DDCR U?
+L TPS563209DDCR U2
 U 1 1 546091FF
 P 4850 3500
-F 0 "U?" H 4550 3850 40  0000 C CNN
+F 0 "U2" H 4550 3850 40  0000 C CNN
 F 1 "TPS563209DDCR" H 5000 3850 40  0000 C CNN
 F 2 "SOT-23" H 4850 3550 35  0000 C CIN
