File: aleftvca.sch (KiCad schematic (older format))
At the start: 12 parts

Commit message: Some work
Parts:
- removed U?: TL074, symbol TL074
- added U?: TL074, symbol TL074
- C? (x2): value C -> 560p
- C?: value C -> 100p
- R? (x3): value R -> 33k
- R? (x2): value R -> 500
Connections:
- net Out: now also U?.8
- net V+: now also U?.4 (V+)
- net V-: now also U?.11 (V-)
- net Vgnd: now also U?.10 (+)
- net at C?.2, IC?.4 (OUT), IC?.5 (OUT)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: now also U?.9 (-)
Changed lines of the file:
@@
 LIBS:c2
 LIBS:c2-cache
-EELAYER 25 0
+EELAYER 24 0
 EELAYER END
 $Descr A4 11693 8268
@@
 P 3850 2900
 F 0 "R?" V 3930 2900 40  0000 C CNN
-F 1 "R" V 3857 2901 40  0000 C CNN
+F 1 "33k" V 3857 2901 40  0000 C CNN
 F 2 "" V 3780 2900 30  0000 C CNN
 F 3 "" H 3850 2900 30  0000 C CNN
@@
 P 4450 3250
 F 0 "R?" V 4530 3250 40  0000 C CNN
-F 1 "R" V 4457 3251 40  0000 C CNN
+F 1 "500" V 4457 3251 40  0000 C CNN
 F 2 "" V 4380 3250 30  0000 C CNN
 F 3 "" H 4450 3250 30  0000 C CNN
@@
 P 4450 3750
 F 0 "C?" H 4450 3850 40  0000 L CNN
-F 1 "C" H 4456 3665 40  0000 L CNN
+F 1 "560p" H 4456 3665 40  0000 L CNN
 F 2 "" H 4488 3600 30  0000 C CNN
 F 3 "" H 4450 3750 60  0000 C CNN
@@
 P 4450 4350
 F 0 "C?" H 4450 4450 40  0000 L CNN
-F 1 "C" H 4456 4265 40  0000 L CNN
+F 1 "560p" H 4456 4265 40  0000 L CNN
 F 2 "" H 4488 4200 30  0000 C CNN
 F 3 "" H 4450 4350 60  0000 C CNN
@@
 P 4450 4850
 F 0 "R?" V 4530 4850 40  0000 C CNN
-F 1 "R" V 4457 4851 40  0000 C CNN
+F 1 "500" V 4457 4851 40  0000 C CNN
 F 2 "" V 4380 4850 30  0000 C CNN
 F 3 "" H 4450 4850 30  0000 C CNN
@@
 P 3850 5200
 F 0 "R?" V 3930 5200 40  0000 C CNN
-F 1 "R" V 3857 5201 40  0000 C CNN
+F 1 "33k" V 3857 5201 40  0000 C CNN
 F 2 "" V 3780 5200 30  0000 C CNN
 F 3 "" H 3850 5200 30  0000 C CNN
@@
 Wire Wire Line
 	2700 2150 2700 3650
+Wire Wire Line
+	5750 4250 6300 4250
+Connection ~ 5750 4250
+Wire Wire Line
+	2700 2150 6700 2150
+Wire Wire Line
+	6700 2150 6700 3750
+Connection ~ 2700 3550
+Wire Wire Line
+	2700 5650 6700 5650
+Wire Wire Line
+	6700 5650 6700 4550
+Connection ~ 2700 4600
+$Comp
+L R R?
+U 1 1 54614448
+P 6300 4650
+F 0 "R?" V 6380 4650 40  0000 C CNN
+F 1 "33k" V 6307 4651 40  0000 C CNN
+F 2 "" V 6230 4650 30  0000 C CNN
+F 3 "" H 6300 4650 30  0000 C CNN
+	1    6300 4650
+	0    1    1    0
+$EndComp
+$Comp
+L C C?
+U 1 1 5461449F
+P 6250 4950
+F 0 "C?" H 6250 5050 40  0000 L CNN
+F 1 "100p" H 6256 4865 40  0000 L CNN
+F 2 "" H 6288 4800 30  0000 C CNN
+F 3 "" H 6250 4950 60  0000 C CNN
+	1    6250 4950
+	0    1    1    0
+$EndComp
+Wire Wire Line
+	6050 4650 5750 4650
+Connection ~ 5750 4650
+Wire Wire Line
+	6050 4950 5750 4950
+Connection ~ 5750 4950
+Wire Wire Line
+	6550 4650 7300 4650
+Wire Wire Line
+	7300 4150 7300 4950
+Wire Wire Line
+	7300 4950 6450 4950
+Connection ~ 7300 4650
+Text HLabel 7550 4150 2    60   Output ~ 0
+Out
+Wire Wire Line
+	7300 4150 7550 4150
 $Comp
 L TL074 U?
-U 1 1 5461422B
+U 3 1 54FF9E5E
 P 6800 4150
 F 0 "U?" H 6850 4350 60  0000 C CNN
@@
 F 2 "" H 6800 4150 60  0000 C CNN
 F 3 "" H 6800 4150 60  0000 C CNN
-	1    6800 4150
-	1    0    0    -1
-$EndComp
-Wire Wire Line
-	5750 4250 6300 4250
-Connection ~ 5750 4250
-Wire Wire Line
-	2700 2150 6700 2150
-Wire Wire Line
-	6700 2150 6700 3750
-Connection ~ 2700 3550
-Wire Wire Line
-	2700 5650 6700 5650
-Wire Wire Line
-	6700 5650 6700 4550
-Connection ~ 2700 4600
-$Comp
-L R R?
-U 1 1 54614448
-P 6300 4650
-F 0 "R?" V 6380 4650 40  0000 C CNN
-F 1 "R" V 6307 4651 40  0000 C CNN
-F 2 "" V 6230 4650 30  0000 C CNN
-F 3 "" H 6300 4650 30  0000 C CNN
-	1    6300 4650
-	0    1    1    0
-$EndComp
-$Comp
-L C C?
-U 1 1 5461449F
-P 6250 4950
-F 0 "C?" H 6250 5050 40  0000 L CNN
-F 1 "C" H 6256 4865 40  0000 L CNN
-F 2 "" H 6288 4800 30  0000 C CNN
-F 3 "" H 6250 4950 60  0000 C CNN
-	1    6250 4950
-	0    1    1    0
-$EndComp
-Wire Wire Line
-	6050 4650 5750 4650
-Connection ~ 5750 4650
-Wire Wire Line
-	6050 4950 5750 4950
-Connection ~ 5750 4950
-Wire Wire Line
-	6550 4650 7300 4650
-Wire Wire Line
-	7300 4150 7300 4950
-Wire Wire Line
-	7300 4950 6450 4950
-Connection ~ 7300 4650
-Text HLabel 7550 4150 2    60   Output ~ 0
-Out
-Wire Wire Line
-	7300 4150 7550 4150
+	3    6800 4150
+	1    0    0    -1
+$EndComp
 $EndSCHEMATC

Commit message: Ready for tapeout
Parts:
- added R25: DNM, symbol R
- gave numbers to parts that had none: 10
Connections:
- net Vgnd: now also R25.1
- net at IC2.1 (MODE): now also R25.2
Changed lines of the file:
@@
 $Descr A4 11693 8268
 encoding utf-8
-Sheet 5 9
+Sheet 5 10
 Title ""
 Date ""
@@
 Ain
 $Comp
-L SSM2164P IC?
+L SSM2164P IC2
 U 1 1 54613A8F
 P 5050 2900
-F 0 "IC?" H 5250 3100 50  0000 L BNN
+F 0 "IC2" H 5250 3100 50  0000 L BNN
 F 1 "SSM2164P" H 5250 2600 50  0000 L BNN
 F 2 "ssm2164-DIL16" H 5050 3050 50  0001 C CNN
@@
 	1    0    0    -1
 $EndComp
-Wire Wire Line
-	4800 2350 5050 2350
-Wire Wire Line
-	5050 2350 5050 2600
-$Comp
-L R R?
+$Comp
+L R R26
 U 1 1 54613B47
 P 3850 2900
-F 0 "R?" V 3930 2900 40  0000 C CNN
+F 0 "R26" V 3930 2900 40  0000 C CNN
 F 1 "33k" V 3857 2901 40  0000 C CNN
 F 2 "" V 3780 2900 30  0000 C CNN
@@
 $EndComp
 $Comp
-L R R?
+L R R28
 U 1 1 54613BC8
 P 4450 3250
-F 0 "R?" V 4530 3250 40  0000 C CNN
+F 0 "R28" V 4530 3250 40  0000 C CNN
 F 1 "500" V 4457 3251 40  0000 C CNN
 F 2 "" V 4380 3250 30  0000 C CNN
@@
 $EndComp
 $Comp
-L C C?
+L C C24
 U 1 1 54613C17
 P 4450 3750
-F 0 "C?" H 4450 3850 40  0000 L CNN
+F 0 "C24" H 4450 3850 40  0000 L CNN
 F 1 "560p" H 4456 3665 40  0000 L CNN
 F 2 "" H 4488 3600 30  0000 C CNN
@@
 Text HLabel 3400 5200 0    60   Input ~ 0
 Bin
-Wire Wire Line
-	3400 2900 3600 2900
-Wire Wire Line
-	4100 2900 4850 2900
-Wire Wire Line
-	4450 3000 4450 2900
-Connection ~ 4450 2900
-Wire Wire Line
-	4450 3500 4450 3550
-$Comp
-L C C?
+$Comp
+L C C25
 U 1 1 54613CF6
 P 4450 4350
-F 0 "C?" H 4450 4450 40  0000 L CNN
+F 0 "C25" H 4450 4450 40  0000 L CNN
 F 1 "560p" H 4456 4265 40  0000 L CNN
 F 2 "" H 4488 4200 30  0000 C CNN
@@
 $EndComp
 $Comp
-L R R?
+L R R29
 U 1 1 54613D2A
 P 4450 4850
-F 0 "R?" V 4530 4850 40  0000 C CNN
+F 0 "R29" V 4530 4850 40  0000 C CNN
 F 1 "500" V 4457 4851 40  0000 C CNN
 F 2 "" V 4380 4850 30  0000 C CNN
@@
 	-1   0    0    1
 $EndComp
-Wire Wire Line
-	4450 4550 4450 4600
-Wire Wire Line
-	4450 3950 4450 4150
-Wire Wire Line
-	4200 4050 6300 4050
-Connection ~ 4450 4050
-$Comp
-L R R?
+$Comp
+L R R27
 U 1 1 54613DDD
 P 3850 5200
-F 0 "R?" V 3930 5200 40  0000 C CNN
+F 0 "R27" V 3930 5200 40  0000 C CNN
 F 1 "33k" V 3857 5201 40  0000 C CNN
 F 2 "" V 3780 5200 30  0000 C CNN
@@
 	0    1    1    0
 $EndComp
-Wire Wire Line
-	4100 5200 4850 5200
-Wire Wire Line
-	4450 5200 4450 5100
-Wire Wire Line
-	3400 5200 3600 5200
-$Comp
-L SSM2164P IC?
+$Comp
+L SSM2164P IC2
 U 2 1 54613ECC
 P 5050 5200
-F 0 "IC?" H 5250 5400 50  0000 L BNN
+F 0 "IC2" H 5250 5400 50  0000 L BNN
 F 1 "SSM2164P" H 5250 4900 50  0000 L BNN
 F 2 "ssm2164-DIL16" H 5050 5350 50  0001 C CNN
@@
 	1    0    0    -1
 $EndComp
-Connection ~ 4450 5200
-Wire Wire Line
-	4800 4750 5050 4750
-Wire Wire Line
-	5050 4750 5050 4900
-Wire Wire Line
-	5550 2900 5750 2900
-Wire Wire Line
-	5750 2900 5750 5200
-Wire Wire Line
-	5750 5200 5550 5200
-$Comp
-L SSM2164P IC?
+$Comp
+L SSM2164P IC2
 U 5 1 54614084
 P 2700 3950
-F 0 "IC?" H 2900 4150 50  0000 L BNN
+F 0 "IC2" H 2900 4150 50  0000 L BNN
 F 1 "SSM2164P" H 2900 3650 50  0000 L BNN
 F 2 "ssm2164-DIL16" H 2700 4100 50  0001 C CNN
@@
 	1    0    0    -1
 $EndComp
-Wire Wire Line
-	4300 4050 4300 4150
-Wire Wire Line
-	4300 4150 3000 4150
-Connection ~ 4300 4050
-Wire Wire Line
-	2650 4600 2700 4600
-Wire Wire Line
-	2700 4450 2700 5650
-Wire Wire Line
-	2550 3550 2700 3550
-Wire Wire Line
-	2700 2150 2700 3650
-Wire Wire Line
-	5750 4250 6300 4250
-Connection ~ 5750 4250
-Wire Wire Line
-	2700 2150 6700 2150
-Wire Wire Line
-	6700 2150 6700 3750
-Connection ~ 2700 3550
-Wire Wire Line
-	2700 5650 6700 5650
-Wire Wire Line
-	6700 5650 6700 4550
-Connection ~ 2700 4600
-$Comp
-L R R?
+$Comp
+L R R30
 U 1 1 54614448
 P 6300 4650
-F 0 "R?" V 6380 4650 40  0000 C CNN
+F 0 "R30" V 6380 4650 40  0000 C CNN
 F 1 "33k" V 6307 4651 40  0000 C CNN
 F 2 "" V 6230 4650 30  0000 C CNN
@@
 $EndComp
 $Comp
-L C C?
+L C C26
 U 1 1 5461449F
 P 6250 4950
-F 0 "C?" H 6250 5050 40  0000 L CNN
+F 0 "C26" H 6250 5050 40  0000 L CNN
 F 1 "100p" H 6256 4865 40  0000 L CNN
 F 2 "" H 6288 4800 30  0000 C CNN
@@
 	0    1    1    0
 $EndComp
-Wire Wire Line
-	6050 4650 5750 4650
-Connection ~ 5750 4650
-Wire Wire Line
-	6050 4950 5750 4950
-Connection ~ 5750 4950
-Wire Wire Line
-	6550 4650 7300 4650
-Wire Wire Line
-	7300 4150 7300 4950
-Wire Wire Line
-	7300 4950 6450 4950
-Connection ~ 7300 4650
 Text HLabel 7550 4150 2    60   Output ~ 0
 Out
-Wire Wire Line
-	7300 4150 7550 4150
-$Comp
-L TL074 U?
+$Comp
+L TL074 U4
 U 3 1 54FF9E5E
 P 6800 4150
-F 0 "U?" H 6850 4350 60  0000 C CNN
+F 0 "U4" H 6850 4350 60  0000 C CNN
 F 1 "TL074" H 6950 3950 50  0000 C CNN
 F 2 "" H 6800 4150 60  0000 C CNN
@@
 	1    0    0    -1
 $EndComp
+$Comp
+L R R25
+U 1 1 55055DE4
+P 3350 3950
+F 0 "R25" V 3430 3950 40  0000 C CNN
+F 1 "DNM" V 3357 3951 40  0000 C CNN
+F 2 "" V 3280 3950 30  0000 C CNN
+F 3 "" H 3350 3950 30  0000 C CNN
+	1    3350 3950
+	0    1    1    0
+$EndComp
+Wire Wire Line
+	4800 2350 5050 2350
+Wire Wire Line
+	5050 2350 5050 2600
+Wire Wire Line
+	3400 2900 3600 2900
+Wire Wire Line
+	4100 2900 4850 2900
+Wire Wire Line
+	4450 3000 4450 2900
+Connection ~ 4450 2900
+Wire Wire Line
+	4450 3500 4450 3550
+Wire Wire Line
+	4450 4550 4450 4600
+Wire Wire Line
+	4450 3950 4450 4150
+Wire Wire Line
+	4200 4050 6300 4050
+Connection ~ 4450 4050
+Wire Wire Line
+	4100 5200 4850 5200
+Wire Wire Line
+	4450 5200 4450 5100
+Wire Wire Line
+	3400 5200 3600 5200
+Connection ~ 4450 5200
+Wire Wire Line
+	4800 4750 5050 4750
+Wire Wire Line
+	5050 4750 5050 4900
+Wire Wire Line
+	5550 2900 5750 2900
+Wire Wire Line
+	5750 2900 5750 5200
+Wire Wire Line
+	5750 5200 5550 5200
+Wire Wire Line
+	4300 4050 4300 4150
+Wire Wire Line
+	4300 4150 3000 4150
+Connection ~ 4300 4050
+Wire Wire Line
+	2650 4600 2700 4600
+Wire Wire Line
+	2700 4450 2700 5650
+Wire Wire Line
+	2550 3550 2700 3550
+Wire Wire Line
+	2700 2150 2700 3650
+Wire Wire Line
+	5750 4250 6300 4250
+Connection ~ 5750 4250
+Wire Wire Line
+	2700 2150 6700 2150
+Wire Wire Line
+	6700 2150 6700 3750
+Connection ~ 2700 3550
+Wire Wire Line
+	2700 5650 6700 5650
+Wire Wire Line
+	6700 5650 6700 4550
+Connection ~ 2700 4600
+Wire Wire Line
+	6050 4650 5750 4650
+Connection ~ 5750 4650
+Wire Wire Line
+	6050 4950 5750 4950
+Connection ~ 5750 4950
+Wire Wire Line
+	6550 4650 7300 4650
+Wire Wire Line
+	7300 4150 7300 4950
+Wire Wire Line
+	7300 4950 6450 4950
+Connection ~ 7300 4650
+Wire Wire Line
+	7300 4150 7550 4150
+Wire Wire Line
+	3000 3950 3100 3950
+Wire Wire Line
+	3600 3950 3700 3950
+Wire Wire Line
+	3700 3950 3700 4150
+Connection ~ 3700 4150
 $EndSCHEMATC
