File: audioin.sch (KiCad schematic (older format))
At the start: 12 parts

Commit message: Some work
Parts:
- removed C? (x4): CP2, symbol CP2
- removed C? (x3): C, symbol C
- removed R? (x3): 1M, symbol R
- added C? (x4): 100nf, symbol C
- added C? (x3): C, symbol C
- added R? (x8): 100k, symbol R
- added R? (x3): 1M, symbol R
- added U? (x4): TL074, symbol TL074
Connections:
- net ALeftIn: now also C?.2; no longer R?.1
- net ALeftOut: now also R?.1, U?.1
- net ARightIn: now also C?.1, C?.2
- net ARightOut: now also R?.1, U?.7
- net BLeftIn: now also C?.1, C?.2
- net BLeftOut: now also R?.1, U?.8
- net BRightIn: now also C?.1, C?.2
- net BRightOut: now also R?.1, U?.14
- net Gnd: now also C?.2, C?.2, C?.2, R?.2, R?.2, R?.2, R?.2, R?.2, R?.2, R?.2
- new net: C?.1, R?.1, U?.3 (+)
- new net: R?.1, R?.2, U?.2 (-)
- new net: C?.1, R?.1, U?.5 (+)
- new net: R?.1, R?.2, U?.6 (-)
- new net: C?.1, R?.1, U?.10 (+)
- new net: R?.1, R?.2, U?.9 (-)
- new net: C?.1, R?.1, U?.12 (+)
- new net: R?.1, R?.2, U?.13 (-)
- new net V+: U?.4 (V+), U?.4 (V+), U?.4 (V+), U?.4 (V+)
- new net V-: U?.11 (V-), U?.11 (V-), U?.11 (V-), U?.11 (V-)
Other:
- moved on the sheet: C?, R?

Commit message: Ready for tapeout
Parts:
- C33, C34, C37, C38: renamed from C?; value C -> 22p
- C35, C36, C39, C40: renamed from C?; value 100nf -> 100n
- gave numbers to parts that had none: 13
Connections:
- net Gnd: no longer C33.2, C34.2, C37.2, C38.2
- net V-: now also C33.2, C34.2, C37.2, C38.2
Other:
- note added: "TVS dioder!"
Changed lines of the file:
@@
 $Descr A4 11693 8268
 encoding utf-8
-Sheet 9 9
+Sheet 9 10
 Title ""
 Date ""
@@
 ALeftIn
 $Comp
-L C C?
+L C C33
 U 1 1 5461D3D7
 P 2050 1700
-F 0 "C?" H 2050 1800 40  0000 L CNN
-F 1 "C" H 2056 1615 40  0000 L CNN
+F 0 "C33" H 2050 1800 40  0000 L CNN
+F 1 "22p" H 2056 1615 40  0000 L CNN
 F 2 "" H 2088 1550 30  0000 C CNN
 F 3 "" H 2050 1700 60  0000 C CNN
@@
 Gnd
 $Comp
-L R R?
+L R R39
 U 1 1 5461D421
 P 2650 1750
-F 0 "R?" V 2730 1750 40  0000 C CNN
+F 0 "R39" V 2730 1750 40  0000 C CNN
 F 1 "1M" V 2657 1751 40  0000 C CNN
 F 2 "" V 2580 1750 30  0000 C CNN
@@
 BRightOut
 $Comp
-L C C?
+L C C35
 U 1 1 54B1187D
 P 2350 1400
-F 0 "C?" H 2350 1500 40  0000 L CNN
-F 1 "100nf" H 2356 1315 40  0000 L CNN
+F 0 "C35" H 2350 1500 40  0000 L CNN
+F 1 "100n" H 2356 1315 40  0000 L CNN
 F 2 "" H 2388 1250 30  0000 C CNN
 F 3 "" H 2350 1400 60  0000 C CNN
@@
 	2550 1400 3500 1400
 Wire Wire Line
-	2650 2000 2650 2100
+	2650 2100 2650 2000
 Wire Wire Line
 	1850 2100 2800 2100
 Wire Wire Line
-	2050 1900 2050 2100
-Connection ~ 2050 2100
-Wire Wire Line
 	1850 1400 2150 1400
 $Comp
-L TL074 U?
+L TL074 U5
 U 1 1 54B1192B
 P 4000 1500
-F 0 "U?" H 4050 1700 60  0000 C CNN
+F 0 "U5" H 4050 1700 60  0000 C CNN
 F 1 "TL074" H 4150 1300 50  0000 C CNN
 F 2 "" H 4000 1500 60  0000 C CNN
@@
 $EndComp
 $Comp
-L R R?
+L R R43
 U 1 1 54B11943
 P 3900 2350
-F 0 "R?" V 3980 2350 40  0000 C CNN
+F 0 "R43" V 3980 2350 40  0000 C CNN
 F 1 "100k" V 3907 2351 40  0000 C CNN
 F 2 "" V 3830 2350 30  0000 C CNN
@@
 	3900 1000 3900 1100
 $Comp
-L R R?
+L R R41
 U 1 1 54B11CC3
 P 3050 2100
-F 0 "R?" V 3130 2100 40  0000 C CNN
+F 0 "R41" V 3130 2100 40  0000 C CNN
 F 1 "100k" V 3057 2101 40  0000 C CNN
 F 2 "" V 2980 2100 30  0000 C CNN
@@
 Connection ~ 4600 1500
 $Comp
-L TL074 U?
+L TL074 U5
 U 2 1 54B11DDC
 P 4000 3300
-F 0 "U?" H 4050 3500 60  0000 C CNN
+F 0 "U5" H 4050 3500 60  0000 C CNN
 F 1 "TL074" H 4150 3100 50  0000 C CNN
 F 2 "" H 4000 3300 60  0000 C CNN
@@
 $EndComp
 $Comp
-L TL074 U?
+L TL074 U5
 U 3 1 54B11DF0
 P 8950 1600
-F 0 "U?" H 9000 1800 60  0000 C CNN
+F 0 "U5" H 9000 1800 60  0000 C CNN
 F 1 "TL074" H 9100 1400 50  0000 C CNN
 F 2 "" H 8950 1600 60  0000 C CNN
@@
 $EndComp
 $Comp
-L TL074 U?
+L TL074 U5
 U 4 1 54B11E04
 P 8950 3350
-F 0 "U?" H 9000 3550 60  0000 C CNN
+F 0 "U5" H 9000 3550 60  0000 C CNN
 F 1 "TL074" H 9100 3150 50  0000 C CNN
 F 2 "" H 8950 3350 60  0000 C CNN
@@
 $EndComp
 $Comp
-L C C?
+L C C34
 U 1 1 54B11E17
 P 2050 3500
-F 0 "C?" H 2050 3600 40  0000 L CNN
-F 1 "C" H 2056 3415 40  0000 L CNN
+F 0 "C34" H 2050 3600 40  0000 L CNN
+F 1 "22p" H 2056 3415 40  0000 L CNN
 F 2 "" H 2088 3350 30  0000 C CNN
 F 3 "" H 2050 3500 60  0000 C CNN
@@
 Gnd
 $Comp
-L R R?
+L R R40
 U 1 1 54B11E1E
 P 2650 3550
-F 0 "R?" V 2730 3550 40  0000 C CNN
+F 0 "R40" V 2730 3550 40  0000 C CNN
 F 1 "1M" V 2657 3551 40  0000 C CNN
 F 2 "" V 2580 3550 30  0000 C CNN
@@
 Connection ~ 2050 3200
 $Comp
-L C C?
+L C C36
 U 1 1 54B11E27
 P 2350 3200
-F 0 "C?" H 2350 3300 40  0000 L CNN
-F 1 "100nf" H 2356 3115 40  0000 L CNN
+F 0 "C36" H 2350 3300 40  0000 L CNN
+F 1 "100n" H 2356 3115 40  0000 L CNN
 F 2 "" H 2388 3050 30  0000 C CNN
 F 3 "" H 2350 3200 60  0000 C CNN
@@
 	2550 3200 3500 3200
 Wire Wire Line
-	2650 3800 2650 3900
+	2650 3900 2650 3800
 Wire Wire Line
 	1850 3900 2800 3900
 Wire Wire Line
-	2050 3700 2050 3900
-Connection ~ 2050 3900
-Wire Wire Line
 	1850 3200 2150 3200
 $Comp
-L R R?
+L R R44
 U 1 1 54B11E3A
 P 3900 4150
-F 0 "R?" V 3980 4150 40  0000 C CNN
+F 0 "R44" V 3980 4150 40  0000 C CNN
 F 1 "100k" V 3907 4151 40  0000 C CNN
 F 2 "" V 3830 4150 30  0000 C CNN
@@
 	3900 2800 3900 2900
 $Comp
-L R R?
+L R R42
 U 1 1 54B11E43
 P 3050 3900
-F 0 "R?" V 3130 3900 40  0000 C CNN
+F 0 "R42" V 3130 3900 40  0000 C CNN
 F 1 "100k" V 3057 3901 40  0000 C CNN
 F 2 "" V 2980 3900 30  0000 C CNN
@@
 Connection ~ 4600 3300
 $Comp
-L C C?
+L C C37
 U 1 1 54B11E58
 P 7000 1800
-F 0 "C?" H 7000 1900 40  0000 L CNN
-F 1 "C" H 7006 1715 40  0000 L CNN
+F 0 "C37" H 7000 1900 40  0000 L CNN
+F 1 "22p" H 7006 1715 40  0000 L CNN
 F 2 "" H 7038 1650 30  0000 C CNN
 F 3 "" H 7000 1800 60  0000 C CNN
@@
 Gnd
 $Comp
-L R R?
+L R R45
 U 1 1 54B11E5F
 P 7600 1850
-F 0 "R?" V 7680 1850 40  0000 C CNN
+F 0 "R45" V 7680 1850 40  0000 C CNN
 F 1 "1M" V 7607 1851 40  0000 C CNN
 F 2 "" V 7530 1850 30  0000 C CNN
@@
 Connection ~ 7000 1500
 $Comp
-L C C?
+L C C39
 U 1 1 54B11E68
 P 7300 1500
-F 0 "C?" H 7300 1600 40  0000 L CNN
-F 1 "100nf" H 7306 1415 40  0000 L CNN
+F 0 "C39" H 7300 1600 40  0000 L CNN
+F 1 "100n" H 7306 1415 40  0000 L CNN
 F 2 "" H 7338 1350 30  0000 C CNN
 F 3 "" H 7300 1500 60  0000 C CNN
@@
 	7500 1500 8450 1500
 Wire Wire Line
-	7600 2100 7600 2200
+	7600 2200 7600 2100
 Wire Wire Line
 	6800 2200 7750 2200
 Wire Wire Line
-	7000 2000 7000 2200
-Connection ~ 7000 2200
-Wire Wire Line
 	6800 1500 7100 1500
 $Comp
-L R R?
+L R R49
 U 1 1 54B11E7B
 P 8850 2450
-F 0 "R?" V 8930 2450 40  0000 C CNN
+F 0 "R49" V 8930 2450 40  0000 C CNN
 F 1 "100k" V 8857 2451 40  0000 C CNN
 F 2 "" V 8780 2450 30  0000 C CNN
@@
 	8850 1100 8850 1200
 $Comp
-L R R?
+L R R47
 U 1 1 54B11E84
 P 8000 2200
-F 0 "R?" V 8080 2200 40  0000 C CNN
+F 0 "R47" V 8080 2200 40  0000 C CNN
 F 1 "100k" V 8007 2201 40  0000 C CNN
 F 2 "" V 7930 2200 30  0000 C CNN
@@
 Connection ~ 9550 1600
 $Comp
-L C C?
+L C C38
 U 1 1 54B11EF5
 P 7000 3550
-F 0 "C?" H 7000 3650 40  0000 L CNN
-F 1 "C" H 7006 3465 40  0000 L CNN
+F 0 "C38" H 7000 3650 40  0000 L CNN
+F 1 "22p" H 7006 3465 40  0000 L CNN
 F 2 "" H 7038 3400 30  0000 C CNN
 F 3 "" H 7000 3550 60  0000 C CNN
@@
 Gnd
 $Comp
-L R R?
+L R R46
 U 1 1 54B11EFC
 P 7600 3600
-F 0 "R?" V 7680 3600 40  0000 C CNN
+F 0 "R46" V 7680 3600 40  0000 C CNN
 F 1 "1M" V 7607 3601 40  0000 C CNN
 F 2 "" V 7530 3600 30  0000 C CNN
@@
 Connection ~ 7000 3250
 $Comp
-L C C?
+L C C40
 U 1 1 54B11F04
 P 7300 3250
-F 0 "C?" H 7300 3350 40  0000 L CNN
-F 1 "100nf" H 7306 3165 40  0000 L CNN
+F 0 "C40" H 7300 3350 40  0000 L CNN
+F 1 "100n" H 7306 3165 40  0000 L CNN
 F 2 "" H 7338 3100 30  0000 C CNN
 F 3 "" H 7300 3250 60  0000 C CNN
@@
 	7500 3250 8450 3250
 Wire Wire Line
-	7600 3850 7600 3950
+	7600 3950 7600 3850
 Wire Wire Line
 	6800 3950 7750 3950
 Wire Wire Line
-	7000 3750 7000 3950
-Connection ~ 7000 3950
-Wire Wire Line
 	6800 3250 7100 3250
 $Comp
-L R R?
+L R R50
 U 1 1 54B11F11
 P 8850 4200
-F 0 "R?" V 8930 4200 40  0000 C CNN
+F 0 "R50" V 8930 4200 40  0000 C CNN
 F 1 "100k" V 8857 4201 40  0000 C CNN
 F 2 "" V 8780 4200 30  0000 C CNN
@@
 	8850 2850 8850 2950
 $Comp
-L R R?
+L R R48
 U 1 1 54B11F1A
 P 8000 3950
-F 0 "R?" V 8080 3950 40  0000 C CNN
+F 0 "R48" V 8080 3950 40  0000 C CNN
 F 1 "100k" V 8007 3951 40  0000 C CNN
 F 2 "" V 7930 3950 30  0000 C CNN
@@
 	8850 3750 8850 3850
 Connection ~ 9550 3350
+Text Notes 1350 2600 0    60   ~ 0
+TVS dioder!
+Text HLabel 2050 2200 3    60   Input ~ 0
+V-
+Wire Wire Line
+	2050 2200 2050 1900
+Text HLabel 2050 4000 3    60   Input ~ 0
+V-
+Wire Wire Line
+	2050 4000 2050 3700
+Text HLabel 7000 4050 3    60   Input ~ 0
+V-
+Wire Wire Line
+	7000 4050 7000 3750
+Text HLabel 7000 2300 3    60   Input ~ 0
+V-
+Wire Wire Line
+	7000 2300 7000 2000
 $EndSCHEMATC
