File: audioout.sch (KiCad schematic (older format))
At the start: 6 parts

Commit message: Ready for tapeout
Parts:
- removed C? (x2): C, symbol C
- gave numbers to parts that had none: 4
Changed lines of the file:
@@
 $Descr A4 11693 8268
 encoding utf-8
-Sheet 8 9
+Sheet 8 10
 Title ""
 Date ""
@@
 GNDPWR
 $Comp
-L CP2 C?
+L CP2 C31
 U 1 1 5462F191
 P 3300 2200
-F 0 "C?" H 3300 2300 40  0000 L CNN
+F 0 "C31" H 3300 2300 40  0000 L CNN
 F 1 "CP2" H 3306 2115 40  0000 L CNN
 F 2 "" H 3338 2050 30  0000 C CNN
@@
 $EndComp
 $Comp
-L CP2 C?
+L CP2 C32
 U 1 1 5462F1F2
 P 3300 2650
-F 0 "C?" H 3300 2750 40  0000 L CNN
+F 0 "C32" H 3300 2750 40  0000 L CNN
 F 1 "CP2" H 3306 2565 40  0000 L CNN
 F 2 "" H 3338 2500 30  0000 C CNN
@@
 	2400 2650 3100 2650
 $Comp
-L R R?
+L R R37
 U 1 1 5462F22F
 P 3700 3050
-F 0 "R?" V 3780 3050 40  0000 C CNN
+F 0 "R37" V 3780 3050 40  0000 C CNN
 F 1 "1M" V 3707 3051 40  0000 C CNN
 F 2 "" V 3630 3050 30  0000 C CNN
@@
 $EndComp
 $Comp
-L R R?
+L R R38
 U 1 1 5462F2A6
 P 4000 3050
-F 0 "R?" V 4080 3050 40  0000 C CNN
+F 0 "R38" V 4080 3050 40  0000 C CNN
 F 1 "1M" V 4007 3051 40  0000 C CNN
 F 2 "" V 3930 3050 30  0000 C CNN
@@
 	3500 2200 5100 2200
 Wire Wire Line
-	2300 3500 4600 3500
+	2300 3500 4000 3500
 Wire Wire Line
 	4000 3500 4000 3300
@@
 Connection ~ 3700 2650
 Connection ~ 4000 2200
-$Comp
-L C C?
-U 1 1 54631C45
-P 4300 3000
-F 0 "C?" H 4300 3100 40  0000 L CNN
-F 1 "C" H 4306 2915 40  0000 L CNN
-F 2 "" H 4338 2850 30  0000 C CNN
-F 3 "" H 4300 3000 60  0000 C CNN
-	1    4300 3000
-	1    0    0    -1
-$EndComp
-$Comp
-L C C?
-U 1 1 54631C94
-P 4600 3000
-F 0 "C?" H 4600 3100 40  0000 L CNN
-F 1 "C" H 4606 2915 40  0000 L CNN
-F 2 "" H 4638 2850 30  0000 C CNN
-F 3 "" H 4600 3000 60  0000 C CNN
-	1    4600 3000
-	1    0    0    -1
-$EndComp
-Wire Wire Line
-	4300 3500 4300 3200
-Connection ~ 4000 3500
-Wire Wire Line
-	4600 3500 4600 3200
-Connection ~ 4300 3500
-Wire Wire Line
-	4300 2800 4300 2650
-Connection ~ 4300 2650
-Wire Wire Line
-	4600 2200 4600 2800
-Connection ~ 4600 2200
 $EndSCHEMATC
