File: powerin.sch (KiCad schematic (older format))
At the start: 5 parts

Commit message: Ready for tapeout
Parts:
- C30: renamed from C?; value C -> 1u
- R36: renamed from R?; value R -> 470
- gave numbers to parts that had none: 3
Changed lines of the file:
@@
 $Descr A4 11693 8268
 encoding utf-8
-Sheet 7 9
+Sheet 7 10
 Title ""
 Date ""
@@
 $EndDescr
 $Comp
-L C C?
+L C C30
 U 1 1 5461FE64
 P 3550 3100
-F 0 "C?" H 3550 3200 40  0000 L CNN
-F 1 "C" H 3556 3015 40  0000 L CNN
+F 0 "C30" H 3550 3200 40  0000 L CNN
+F 1 "1u" H 3556 3015 40  0000 L CNN
 F 2 "" H 3588 2950 30  0000 C CNN
 F 3 "" H 3550 3100 60  0000 C CNN
@@
 $EndComp
 $Comp
-L FUSE F?
+L FUSE F1
 U 1 1 5461FEF7
 P 2650 2850
-F 0 "F?" H 2750 2900 40  0000 C CNN
+F 0 "F1" H 2750 2900 40  0000 C CNN
 F 1 "FUSE" H 2550 2800 40  0000 C CNN
 F 2 "" H 2650 2850 60  0000 C CNN
@@
 Vin-
 $Comp
-L TVS D?
+L TVS D5
 U 1 1 5461FF78
 P 3150 3200
-F 0 "D?" H 3150 3350 60  0000 C CNN
+F 0 "D5" H 3150 3350 60  0000 C CNN
 F 1 "TVS" H 3150 3050 60  0000 C CNN
 F 2 "" H 3150 3200 60  0000 C CNN
@@
 Connection ~ 3550 2850
 $Comp
-L LED D?
+L LED D6
 U 1 1 546202A4
 P 3950 3100
-F 0 "D?" H 3950 3200 50  0000 C CNN
+F 0 "D6" H 3950 3200 50  0000 C CNN
 F 1 "LED" H 3950 3000 50  0000 C CNN
 F 2 "" H 3950 3100 60  0000 C CNN
@@
 Connection ~ 3950 2850
 $Comp
-L R R?
+L R R36
 U 1 1 54620343
 P 3950 3600
-F 0 "R?" V 4030 3600 40  0000 C CNN
-F 1 "R" V 3957 3601 40  0000 C CNN
+F 0 "R36" V 4030 3600 40  0000 C CNN
+F 1 "470" V 3957 3601 40  0000 C CNN
 F 2 "" V 3880 3600 30  0000 C CNN
 F 3 "" H 3950 3600 30  0000 C CNN
