File: rightvca.sch (KiCad schematic (older format))
At the start: 11 parts

Commit message: Some work
Parts:
- removed U?: TL074, symbol TL074
- added U?: TL074, symbol TL074
- C? (x2): value C -> 560p
- C?: value C -> 100p
- R? (x3): value R -> 33k
- R? (x2): value R -> 500
Connections:
- net Out: now also U?.14
- net V+: now also U?.4 (V+)
- net V-: now also U?.11 (V-)
- net Vgnd: now also U?.12 (+)
- net at C?.2, IC?.12 (OUT), IC?.13 (OUT)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: now also U?.13 (-)
Changed lines of the file:
@@
 LIBS:c2
 LIBS:c2-cache
-EELAYER 25 0
+EELAYER 24 0
 EELAYER END
 $Descr A4 11693 8268
@@
 P 3900 2550
 F 0 "R?" V 3980 2550 40  0000 C CNN
-F 1 "R" V 3907 2551 40  0000 C CNN
+F 1 "33k" V 3907 2551 40  0000 C CNN
 F 2 "" V 3830 2550 30  0000 C CNN
 F 3 "" H 3900 2550 30  0000 C CNN
@@
 P 4500 2900
 F 0 "R?" V 4580 2900 40  0000 C CNN
-F 1 "R" V 4507 2901 40  0000 C CNN
+F 1 "500" V 4507 2901 40  0000 C CNN
 F 2 "" V 4430 2900 30  0000 C CNN
 F 3 "" H 4500 2900 30  0000 C CNN
@@
 P 4500 3400
 F 0 "C?" H 4500 3500 40  0000 L CNN
-F 1 "C" H 4506 3315 40  0000 L CNN
+F 1 "560p" H 4506 3315 40  0000 L CNN
 F 2 "" H 4538 3250 30  0000 C CNN
 F 3 "" H 4500 3400 60  0000 C CNN
@@
 P 4500 4000
 F 0 "C?" H 4500 4100 40  0000 L CNN
-F 1 "C" H 4506 3915 40  0000 L CNN
+F 1 "560p" H 4506 3915 40  0000 L CNN
 F 2 "" H 4538 3850 30  0000 C CNN
 F 3 "" H 4500 4000 60  0000 C CNN
@@
 P 4500 4500
 F 0 "R?" V 4580 4500 40  0000 C CNN
-F 1 "R" V 4507 4501 40  0000 C CNN
+F 1 "500" V 4507 4501 40  0000 C CNN
 F 2 "" V 4430 4500 30  0000 C CNN
 F 3 "" H 4500 4500 30  0000 C CNN
@@
 P 3900 4850
 F 0 "R?" V 3980 4850 40  0000 C CNN
-F 1 "R" V 3907 4851 40  0000 C CNN
+F 1 "33k" V 3907 4851 40  0000 C CNN
 F 2 "" V 3830 4850 30  0000 C CNN
 F 3 "" H 3900 4850 30  0000 C CNN
@@
 Wire Wire Line
 	5800 4850 5600 4850
-$Comp
-L TL074 U?
-U 1 1 54616C7C
-P 6850 3800
-F 0 "U?" H 6900 4000 60  0000 C CNN
-F 1 "TL074" H 7000 3600 50  0000 C CNN
-F 2 "" H 6850 3800 60  0000 C CNN
-F 3 "" H 6850 3800 60  0000 C CNN
-	1    6850 3800
-	1    0    0    -1
-$EndComp
 Wire Wire Line
 	5800 3900 6350 3900
@@
 P 6350 4300
 F 0 "R?" V 6430 4300 40  0000 C CNN
-F 1 "R" V 6357 4301 40  0000 C CNN
+F 1 "33k" V 6357 4301 40  0000 C CNN
 F 2 "" V 6280 4300 30  0000 C CNN
 F 3 "" H 6350 4300 30  0000 C CNN
@@
 P 6300 4600
 F 0 "C?" H 6300 4700 40  0000 L CNN
-F 1 "C" H 6306 4515 40  0000 L CNN
+F 1 "100p" H 6306 4515 40  0000 L CNN
 F 2 "" H 6338 4450 30  0000 C CNN
 F 3 "" H 6300 4600 60  0000 C CNN
@@
 	1    0    0    -1
 $EndComp
+$Comp
+L TL074 U?
+U 4 1 54FF9F9C
+P 6850 3800
+F 0 "U?" H 6900 4000 60  0000 C CNN
+F 1 "TL074" H 7000 3600 50  0000 C CNN
+F 2 "" H 6850 3800 60  0000 C CNN
+F 3 "" H 6850 3800 60  0000 C CNN
+	4    6850 3800
+	1    0    0    -1
+$EndComp

Commit message: Ready for tapeout
Parts:
- gave numbers to parts that had none: 10
Changed lines of the file:
@@
 $Descr A4 11693 8268
 encoding utf-8
-Sheet 6 9
+Sheet 6 10
 Title ""
 Date ""
@@
 	5100 2000 5100 2250
 $Comp
-L R R?
+L R R31
 U 1 1 54616C2A
 P 3900 2550
-F 0 "R?" V 3980 2550 40  0000 C CNN
+F 0 "R31" V 3980 2550 40  0000 C CNN
 F 1 "33k" V 3907 2551 40  0000 C CNN
 F 2 "" V 3830 2550 30  0000 C CNN
@@
 $EndComp
 $Comp
-L R R?
+L R R33
 U 1 1 54616C31
 P 4500 2900
-F 0 "R?" V 4580 2900 40  0000 C CNN
+F 0 "R33" V 4580 2900 40  0000 C CNN
 F 1 "500" V 4507 2901 40  0000 C CNN
 F 2 "" V 4430 2900 30  0000 C CNN
@@
 $EndComp
 $Comp
-L C C?
+L C C27
 U 1 1 54616C38
 P 4500 3400
-F 0 "C?" H 4500 3500 40  0000 L CNN
+F 0 "C27" H 4500 3500 40  0000 L CNN
 F 1 "560p" H 4506 3315 40  0000 L CNN
 F 2 "" H 4538 3250 30  0000 C CNN
@@
 	4500 3150 4500 3200
 $Comp
-L C C?
+L C C28
 U 1 1 54616C45
 P 4500 4000
-F 0 "C?" H 4500 4100 40  0000 L CNN
+F 0 "C28" H 4500 4100 40  0000 L CNN
 F 1 "560p" H 4506 3915 40  0000 L CNN
 F 2 "" H 4538 3850 30  0000 C CNN
@@
 $EndComp
 $Comp
-L R R?
+L R R34
 U 1 1 54616C4C
 P 4500 4500
-F 0 "R?" V 4580 4500 40  0000 C CNN
+F 0 "R34" V 4580 4500 40  0000 C CNN
 F 1 "500" V 4507 4501 40  0000 C CNN
 F 2 "" V 4430 4500 30  0000 C CNN
@@
 Connection ~ 4500 3700
 $Comp
-L R R?
+L R R32
 U 1 1 54616C57
 P 3900 4850
-F 0 "R?" V 3980 4850 40  0000 C CNN
+F 0 "R32" V 3980 4850 40  0000 C CNN
 F 1 "33k" V 3907 4851 40  0000 C CNN
 F 2 "" V 3830 4850 30  0000 C CNN
@@
 	6750 5300 6750 4200
 $Comp
-L R R?
+L R R35
 U 1 1 54616C8B
 P 6350 4300
-F 0 "R?" V 6430 4300 40  0000 C CNN
+F 0 "R35" V 6430 4300 40  0000 C CNN
 F 1 "33k" V 6357 4301 40  0000 C CNN
 F 2 "" V 6280 4300 30  0000 C CNN
@@
 $EndComp
 $Comp
-L C C?
+L C C29
 U 1 1 54616C92
 P 6300 4600
-F 0 "C?" H 6300 4700 40  0000 L CNN
+F 0 "C29" H 6300 4700 40  0000 L CNN
 F 1 "100p" H 6306 4515 40  0000 L CNN
 F 2 "" H 6338 4450 30  0000 C CNN
@@
 	7350 3800 7600 3800
 $Comp
-L SSM2164P IC?
+L SSM2164P IC2
 U 3 1 54616F08
 P 5100 2550
-F 0 "IC?" H 5300 2750 50  0000 L BNN
+F 0 "IC2" H 5300 2750 50  0000 L BNN
 F 1 "SSM2164P" H 5300 2250 50  0000 L BNN
 F 2 "ssm2164-DIL16" H 5100 2700 50  0001 C CNN
@@
 $EndComp
 $Comp
-L SSM2164P IC?
+L SSM2164P IC2
 U 4 1 54616F77
 P 5100 4850
-F 0 "IC?" H 5300 5050 50  0000 L BNN
+F 0 "IC2" H 5300 5050 50  0000 L BNN
 F 1 "SSM2164P" H 5300 4550 50  0000 L BNN
 F 2 "ssm2164-DIL16" H 5100 5000 50  0001 C CNN
@@
 $EndComp
 $Comp
-L TL074 U?
+L TL074 U4
 U 4 1 54FF9F9C
 P 6850 3800
-F 0 "U?" H 6900 4000 60  0000 C CNN
+F 0 "U4" H 6900 4000 60  0000 C CNN
 F 1 "TL074" H 7000 3600 50  0000 C CNN
 F 2 "" H 6850 3800 60  0000 C CNN
